File: kicad/telegram-doorman.kicad_sch (KiCad schematic)
At the start: 23 parts, among them J1 Conn_01x03_Pin, J2 Conn_01x02_Pin, J3 Conn_01x02_Pin, J4 Conn_01x02_Pin, Q1 2N3904, U1 WeMos_D1_mini, U2 LM393, U3 PC817, U4 PC817, U5 TSR_1-2450

Commit message: add ota, fix door open notif,
Connections:
- net GND: now also U2.5 (+), U2.6 (-), U2.7
Other:
- note added: "Jumper Plug Connected: D1 mini power from TCS:BUS P-Line Not Connected: D1 mini power from external"
- note added: "Jumper Plug Connected: Reset to Default Settings Not Connected: Load Config from Saved"
- note added: "TCS:BUS RX"
- note added: "TCS:BUS TX"
- note removed: "Jumper Plug Connected: D1 mini power from TCS P-Line Not Connected: D1 mini power from 5V"
- note removed: "Jumper Plug Connected: Reset to Factory Settings Not Connected: Load Config from FS"
- note removed: "TCS BUS RX"
- note removed: "TCS BUS TX"
- moved on the sheet: U2B
Changed lines of the file:
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@@
 	)
 	(junction
+		(at 41.91 139.7)
+		(diameter 0)
+		(color 0 0 0 0)
+	)
+	(junction
 		(at 110.49 120.65)
 		(diameter 0)
@@
 	(wire
 		(pts
+			(xy 59.69 137.16) (xy 59.69 138.43)
+		)
+		(stroke
+			(width 0)
+			(type default)
+		)
+	)
+	(wire
+		(pts
 			(xy 105.41 64.77) (xy 109.22 64.77)
 		)
@@
 	(wire
 		(pts
+			(xy 41.91 139.7) (xy 43.18 139.7)
+		)
+		(stroke
+			(width 0)
+			(type default)
+		)
+	)
+	(wire
+		(pts
 			(xy 152.4 123.19) (xy 156.21 123.19)
 		)
@@
 	(wire
 		(pts
+			(xy 41.91 134.62) (xy 41.91 139.7)
+		)
+		(stroke
+			(width 0)
+			(type default)
+		)
+	)
+	(wire
+		(pts
 			(xy 156.21 102.87) (xy 156.21 106.68)
 		)
@@
 	(wire
 		(pts
+			(xy 41.91 139.7) (xy 41.91 140.97)
+		)
+		(stroke
+			(width 0)
+			(type default)
+		)
+	)
+	(wire
+		(pts
 			(xy 36.83 76.2) (xy 45.72 76.2)
 		)
@@
 	(wire
 		(pts
+			(xy 58.42 137.16) (xy 59.69 137.16)
+		)
+		(stroke
+			(width 0)
+			(type default)
+		)
+	)
+	(wire
+		(pts
 			(xy 110.49 120.65) (xy 119.38 120.65)
 		)
@@
 	(wire
 		(pts
+			(xy 43.18 134.62) (xy 41.91 134.62)
+		)
+		(stroke
+			(width 0)
+			(type default)
+		)
+	)
+	(wire
+		(pts
 			(xy 41.91 31.75) (xy 39.37 31.75)
 		)
@@
 		)
 	)
-	(text "TCS BUS TX"
+	(text "TCS:BUS TX"
 		(exclude_from_sim no)
 		(at 191.008 94.234 0)
@@
 		)
 	)
-	(text "TCS BUS RX"
+	(text "TCS:BUS RX"
 		(exclude_from_sim no)
 		(at 87.884 94.234 0)
@@
 		)
 	)
-	(text "Jumper Plug\nConnected: Reset to Factory Settings\nNot Connected: Load Config from FS"
+	(text "Jumper Plug\nConnected: Reset to Default Settings\nNot Connected: Load Config from Saved"
 		(exclude_from_sim no)
 		(at 24.13 96.52 0)
@@
 		)
 	)
-	(text "Jumper Plug\nConnected: D1 mini power from TCS P-Line\nNot Connected: D1 mini power from 5V"
+	(text "Jumper Plug\nConnected: D1 mini power from TCS:BUS P-Line\nNot Connected: D1 mini power from external "
 		(exclude_from_sim no)
 		(at 22.86 51.054 0)
@@
 	(symbol
 		(lib_id "Comparator:LM393")
-		(at 48.26 138.43 0)
+		(at 50.8 137.16 0)
 		(unit 2)
 		(exclude_from_sim no)
@@
 		(fields_autoplaced yes)
 		(property "Reference" "U2"
-			(at 48.26 128.27 0)
+			(at 50.8 127 0)
 			(effects
 				(font
@@
 		)
 		(property "Value" "LM393"
-			(at 48.26 130.81 0)
+			(at 50.8 129.54 0)
 			(effects
 				(font
@@
 		)
 		(property "Footprint" ""
-			(at 48.26 138.43 0)
+			(at 50.8 137.16 0)
 			(effects
 				(font
@@
 		)
 		(property "Datasheet" "http://www.ti.com/lit/ds/symlink/lm393.pdf"
-			(at 48.26 138.43 0)
+			(at 50.8 137.16 0)
 			(effects
 				(font
@@
 		)
 		(property "Description" "Low-Power, Low-Offset Voltage, Dual Comparators, DIP-8/SOIC-8/TO-99-8"
-			(at 48.26 138.43 0)
+			(at 50.8 137.16 0)
 			(effects
 				(font
@@
 	(symbol
 		(lib_id "power:GND")
+		(at 59.69 138.43 0)
+		(unit 1)
+		(exclude_from_sim no)
+		(in_bom yes)
+		(on_board yes)
+		(dnp no)
+		(fields_autoplaced yes)
+		(property "Reference" "#PWR02"
+			(at 59.69 144.78 0)
+			(effects
+				(font
+					(size 1.27 1.27)
+				)
+				(hide yes)
+			)
+		)
+		(property "Value" "GND"
+			(at 59.69 143.51 0)
+			(effects
+				(font
+					(size 1.27 1.27)
+				)
+			)
+		)
+		(property "Footprint" ""
+			(at 59.69 138.43 0)
+			(effects
+				(font
+					(size 1.27 1.27)
+				)
+				(hide yes)
+			)
+		)
+		(property "Datasheet" ""
+			(at 59.69 138.43 0)
+			(effects
+				(font
+					(size 1.27 1.27)
+				)
+				(hide yes)
+			)
+		)
+		(property "Description" "Power symbol creates a global label with name \"GND\" , ground"
+			(at 59.69 138.43 0)
+			(effects
+				(font
+					(size 1.27 1.27)
+				)
+				(hide yes)
+			)
+		)
+		(pin "1"
+		)
+		(instances
+			(project "telegram-doorman"
+				(path "/b97eec34-f621-4ba5-b156-42fdf1b954b4"
+					(reference "#PWR02")
+					(unit 1)
+				)
+			)
+		)
+	)
+	(symbol
+		(lib_id "power:GND")
 		(at 43.18 80.01 0)
 		(unit 1)
@@
 					(unit 1)
 				)
+			)
+		)
+	)
+	(symbol
+		(lib_id "power:GND")
+		(at 41.91 140.97 0)
+		(unit 1)
+		(exclude_from_sim no)
+		(in_bom yes)
+		(on_board yes)
+		(dnp no)
+		(fields_autoplaced yes)
+		(property "Reference" "#PWR011"
+			(at 41.91 147.32 0)
+			(effects
+				(font
+					(size 1.27 1.27)
+				)
+				(hide yes)
+			)
+		)
+		(property "Value" "GND"
+			(at 41.91 146.05 0)
+			(effects
+				(font
+					(size 1.27 1.27)
+				)
+			)
+		)
+		(property "Footprint" ""
+			(at 41.91 140.97 0)
+			(effects
+				(font
+					(size 1.27 1.27)
+				)
+				(hide yes)
+			)
+		)
+		(property "Datasheet" ""
+			(at 41.91 140.97 0)
+			(effects
+				(font
+					(size 1.27 1.27)
+				)
+				(hide yes)
+			)
+		)
+		(property "Description" "Power symbol creates a global label with name \"GND\" , ground"
+			(at 41.91 140.97 0)
+			(effects
+				(font
+					(size 1.27 1.27)
+				)
+				(hide yes)
+			)
+		)
+		(pin "1"
+		)
+		(instances
+			(project "telegram-doorman"
+				(path "/b97eec34-f621-4ba5-b156-42fdf1b954b4"
+					(reference "#PWR011")
+					(unit 1)
+				)
